File: Mosfet_rectifier/Mosfet_rectifier.kicad_sch (KiCad schematic)
At the start: 17 parts, among them J1 Conn_01x03, J2 Conn_01x02, U1 LT4320xDD-1, U2 LT4320xDD-1, U3 LT4320xDD-1

Commit message: finished pcb schematic
Parts:
- added C1, C2, C3: C, symbol Device:C
- added Q1, Q2, Q3, Q4, Q5, Q6: BSC052N08NS5, Package_TO_SOT_SMD:TDSON-8-1, symbol Transistor_FET:BSC052N08NS5
- renumbered D3 to D6, D6 to D9
Connections:
- net GND: now also J2.2 (Pin_2), C1.1, C2.1, C3.1, Q1.1 (S), Q1.2 (S), Q1.3 (S), Q3.1 (S), Q3.2 (S), Q3.3 (S), Q5.1 (S), Q5.2 (S), Q5.3 (S); no longer J2.1 (Pin_1)
- net V1: now also Q1.5 (D)
- net V2: now also Q3.5 (D)
- net V3: now also Q5.5 (D)
- net Vout: now also J2.1 (Pin_1), U1.6 (OUTP), U2.6 (OUTP), C1.2, C2.2, C3.2, Q2.5 (D), Q4.5 (D), Q6.5 (D); no longer J2.2 (Pin_2)
- net at U1.3 (BG2): now also Q1.4 (G)
- net at U1.7 (TG1): now also Q2.4 (G)
- net at U1.8 (IN1): now also Q2.1 (S), Q2.2 (S), Q2.3 (S)
- net at U3.3 (BG2): now also Q5.4 (G)
- net at U3.7 (TG1): now also Q6.4 (G)
- net at U3.8 (IN1): now also Q6.1 (S), Q6.2 (S), Q6.3 (S)
- net at U2.3 (BG2): now also Q3.4 (G)
- net at U2.7 (TG1): now also Q4.4 (G)
- net at U2.8 (IN1): now also Q4.1 (S), Q4.2 (S), Q4.3 (S)
Other:
- moved on the sheet: D2, J1, J2, R2
