File: bettermosfetrectifier/better.kicad_sch (KiCad schematic)
At the start: 20 parts, among them IC1 LT4322RMS8#PBF, IC2 LT4322RMS8#PBF, IC3 LT4322RMS8#PBF, IC4 LT4322RMS8#PBF, IC5 LT4322RMS8#PBF, IC6 LT4322RMS8#PBF, J1 Conn_01x02, J2 Conn_01x03, Q1 IRFS7430-7P, Q2 IRFS7430-7P, Q3 IRFS7430-7P, Q4 IRFS7430-7P, Q5 IRFS7430-7P, Q6 IRFS7430-7P

Commit message: Add files via upload
Added depletion mode mosfets and added capacitors on power mosfet gates
Parts:
- added C1, C2, C3, C4, C5, C6: 10nF, Capacitor_SMD:C_0603_1608Metric, symbol Device:C_Small
- added Q10, Q11, Q12, Q7, Q8, Q9: DN3135, Library:SOT-89_3MC_MCH, symbol Library:DN3135
- CVDDA1, CVDDA2, CVDDA3, CVDDA4, CVDDA5, CVDDA6: footprint Capacitor_SMD:C_0201_0603Metric -> Capacitor_SMD:C_0603_1608Metric
Connections:
- net at CVDDA5.1, J2.3 (Pin_3), Q5.2 (SOURCE)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: now also C5.2, Q12.2 (D); no longer IC6.5 (VDDC), IC6.8 (CATHODE)
- net at CVDDA5.2, IC5.4 (VDDA): now also Q9.1 (G)
- net at IC6.1 (GATE), Q6.1 (GATE): now also C6.2
- net at CVDDA6.2, IC6.4 (VDDA): now also Q12.1 (G)
- net at CVDDA3.1, J2.2 (Pin_2), Q3.2 (SOURCE)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: now also C3.2, Q11.2 (D); no longer IC4.5 (VDDC), IC4.8 (CATHODE)
- net at CVDDA3.2, IC3.4 (VDDA): now also Q8.1 (G)
- net at IC3.1 (GATE), Q3.1 (GATE): now also C3.1
- net at IC4.1 (GATE), Q4.1 (GATE): now also C4.2
- net at CVDDA1.1, CVDDA4.1, CVDDA6.1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: now also C2.1, C4.1, C6.1
- net at IC1.1 (GATE), Q1.1 (GATE): now also C2.2
- net at CVDDA1.2, IC1.4 (VDDA): now also Q10.1 (G)
- net at CVDDA2.1, J2.1 (Pin_1), Q1.4 (DRAIN)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: now also C1.2, Q10.2 (D); no longer IC1.5 (VDDC), IC1.8 (CATHODE)
- net at CVDDA4.2, IC4.4 (VDDA): now also Q11.1 (G)
- net at IC5.1 (GATE), Q5.1 (GATE): now also C5.1
- net at CVDDA2.2, IC2.4 (VDDA): now also Q7.1 (G)
- net at IC2.1 (GATE), Q2.1 (GATE): now also C1.1
- new net: J1.1 (Pin_1), Q2.4 (DRAIN), Q3.4 (DRAIN), Q5.4 (DRAIN), Q7.2 (D), Q8.2 (D), Q9.2 (D)
- new net: IC2.5 (VDDC), IC2.8 (CATHODE), Q7.3 (S)
- new net: IC6.5 (VDDC), IC6.8 (CATHODE), Q12.3 (S)
- new net: IC3.5 (VDDC), IC3.8 (CATHODE), Q8.3 (S)
- new net: IC1.5 (VDDC), IC1.8 (CATHODE), Q10.3 (S)
- new net: IC4.5 (VDDC), IC4.8 (CATHODE), Q11.3 (S)
- new net: IC5.5 (VDDC), IC5.8 (CATHODE), Q9.3 (S)

Commit message: Goon
Changed mosfets to 100V 16A ones (old ones were 40V 240A), added footprints to capacitors and terminals
Parts:
- removed Q1, Q2, Q3, Q4, Q5, Q6: IRFS7430-7P, TO127P1524X508-8_7N-V1:TO127P1524X508-8_7N, symbol IRFS7430-7P:IRFS7430-7P
- added H1, H2, H3, H4: MountingHole, MountingHole:MountingHole_3.2mm_M3, symbol Mechanical:MountingHole
- added Q13, Q14, Q16, Q17, Q18, Q19: BSC050N10NS5ATMA1, Package_TO_SOT_SMD:TDSON-8-1, symbol Transistor_FET:BSC13DN30NSFD
- CVDDA1, CVDDA2, CVDDA3, CVDDA4, CVDDA5, CVDDA6: footprint Capacitor_SMD:C_0603_1608Metric -> Capacitor_SMD:C_1210_3225Metric
- J1: footprint Connector:Tag-Connect_TC2030-IDC-FP_2x03_P1.27mm_Vertical -> TerminalBlock:TerminalBlock_MaiXu_MX126-5.0-03P_1x03_P5.00mm
- J2: footprint Connector:Tag-Connect_TC2030-IDC-NL_2x03_P1.27mm_Vertical -> TerminalBlock:TerminalBlock_MaiXu_MX126-5.0-02P_1x02_P5.00mm
Connections:
- net at J1.1 (Pin_1), Q7.2 (D), Q8.2 (D)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: now also Q13.5 (D), Q16.5 (D), Q18.5 (D)
- net at C5.2, CVDDA5.1, J2.3 (Pin_3)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: now also IC5.2 (VSSA), IC5.3 (ANODE), Q18.1 (S), Q18.2 (S), Q18.3 (S), Q19.5 (D)
- net at C6.2, IC6.1 (GATE): now also Q19.4 (G)
- net at IC6.2 (VSSA), IC6.3 (ANODE): now also C2.1, C4.1, C6.1, CVDDA1.1, CVDDA4.1, CVDDA6.1, IC1.2 (VSSA), IC1.3 (ANODE), IC4.2 (VSSA), IC4.3 (ANODE), J1.2 (Pin_2), Q14.1 (S), Q14.2 (S), Q14.3 (S), Q17.1 (S), Q17.2 (S), Q17.3 (S), Q19.1 (S), Q19.2 (S), Q19.3 (S)
- net at C3.2, CVDDA3.1, J2.2 (Pin_2)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: now also IC3.2 (VSSA), IC3.3 (ANODE), Q16.1 (S), Q16.2 (S), Q16.3 (S), Q17.5 (D)
- net at C3.1, IC3.1 (GATE): now also Q16.4 (G)
- net at C4.2, IC4.1 (GATE): now also Q17.4 (G)
- net at C2.2, IC1.1 (GATE): now also Q14.4 (G)
- net at C1.1, IC2.1 (GATE): now also Q13.4 (G)
- net at C1.2, CVDDA2.1, J2.1 (Pin_1)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: now also IC2.2 (VSSA), IC2.3 (ANODE), Q13.1 (S), Q13.2 (S), Q13.3 (S), Q14.5 (D)
- net at C5.1, IC5.1 (GATE): now also Q18.4 (G)
Other:
- moved on the sheet: C1, C2, C3, C4, C5, C6, CVDDA1, CVDDA2, CVDDA3, CVDDA4, CVDDA5, CVDDA6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

Commit message: Add more capacitance
Parts:
- added C10, C11, C12, C7, C8, C9: 220uF, symbol Device:C_Polarized_Small
- CVDDA1, CVDDA2, CVDDA3, CVDDA4, CVDDA5, CVDDA6: value 10uF -> 0.1uF; footprint Capacitor_SMD:C_1210_3225Metric -> Capacitor_SMD:C_0603_1608Metric
- J1: footprint TerminalBlock:TerminalBlock_MaiXu_MX126-5.0-03P_1x03_P5.00mm -> TerminalBlock:TerminalBlock_MaiXu_MX126-5.0-02P_1x02_P5.00mm
- J2: footprint TerminalBlock:TerminalBlock_MaiXu_MX126-5.0-02P_1x02_P5.00mm -> TerminalBlock:TerminalBlock_MaiXu_MX126-5.0-03P_1x03_P5.00mm
Connections:
- net at CVDDA2.2, IC2.4 (VDDA), Q7.1 (G): now also C8.1
- net at C5.2, CVDDA5.1, IC5.2 (VSSA)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: now also C11.2
- net at CVDDA5.2, IC5.4 (VDDA), Q9.1 (G): now also C11.1
- net GND: now reaches C2.1, C4.1, C6.1, CVDDA1.1, CVDDA4.1, CVDDA6.1, IC1.2 (VSSA), IC1.3 (ANODE), IC4.2 (VSSA), IC4.3 (ANODE), IC6.2 (VSSA), IC6.3 (ANODE), J1.2 (Pin_2), Q14.1 (S), Q14.2 (S), Q14.3 (S), Q17.1 (S), Q17.2 (S), Q17.3 (S), Q19.1 (S), Q19.2 (S), Q19.3 (S)
- net GND: now also C10.2, C12.2, C9.2
- net at CVDDA6.2, IC6.4 (VDDA), Q12.1 (G): now also C12.1
- net at C1.2, CVDDA2.1, IC2.2 (VSSA)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: now also C8.2
- net at C3.2, CVDDA3.1, IC3.2 (VSSA)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: now also C7.2
- net at CVDDA3.2, IC3.4 (VDDA), Q8.1 (G): now also C7.1
- net at CVDDA1.2, IC1.4 (VDDA), Q10.1 (G): now also C9.1
- net at CVDDA4.2, IC4.4 (VDDA), Q11.1 (G): now also C10.1

Commit message: made stupid chopped layout :( :( :(
Parts:
- C10, C11, C12, C7, C8, C9: footprint (none) -> Capacitor_SMD:CP_Elec_6.3x5.4_Nichicon
Changed lines of the file:
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@@
 			)
 		)
-		(property "Footprint" ""
+		(property "Footprint" "Capacitor_SMD:CP_Elec_6.3x5.4_Nichicon"
 			(at 124.46 45.72 0)
 			(hide yes)
@@
 			)
 		)
-		(property "Footprint" ""
+		(property "Footprint" "Capacitor_SMD:CP_Elec_6.3x5.4_Nichicon"
 			(at 123.19 100.33 0)
 			(hide yes)
@@
 			)
 		)
-		(property "Footprint" ""
+		(property "Footprint" "Capacitor_SMD:CP_Elec_6.3x5.4_Nichicon"
 			(at 124.46 156.21 0)
 			(hide yes)
@@
 			)
 		)
-		(property "Footprint" ""
+		(property "Footprint" "Capacitor_SMD:CP_Elec_6.3x5.4_Nichicon"
 			(at 83.82 49.53 0)
 			(hide yes)
@@
 			)
 		)
-		(property "Footprint" ""
+		(property "Footprint" "Capacitor_SMD:CP_Elec_6.3x5.4_Nichicon"
 			(at 83.82 104.14 0)
 			(hide yes)
@@
 			)
 		)
-		(property "Footprint" ""
+		(property "Footprint" "Capacitor_SMD:CP_Elec_6.3x5.4_Nichicon"
 			(at 77.47 157.48 0)
 			(hide yes)

Commit message: idk improved layout a bit
Parts:
- Q10, Q11, Q12, Q7, Q8, Q9: footprint Library:SOT-89_3MC_MCH -> Package_TO_SOT_SMD:SOT-89-3
Changed lines of the file:
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@@
 			)
 		)
-		(property "Footprint" "Library:SOT-89_3MC_MCH"
+		(property "Footprint" "Package_TO_SOT_SMD:SOT-89-3"
 			(at 132.08 30.48 0)
 			(hide yes)
@@
 			)
 		)
-		(property "Footprint" "Library:SOT-89_3MC_MCH"
+		(property "Footprint" "Package_TO_SOT_SMD:SOT-89-3"
 			(at 132.08 139.7 0)
 			(hide yes)
@@
 			)
 		)
-		(property "Footprint" "Library:SOT-89_3MC_MCH"
+		(property "Footprint" "Package_TO_SOT_SMD:SOT-89-3"
 			(at 69.85 115.57 0)
 			(hide yes)
@@
 			)
 		)
-		(property "Footprint" "Library:SOT-89_3MC_MCH"
+		(property "Footprint" "Package_TO_SOT_SMD:SOT-89-3"
 			(at 72.39 60.96 0)
 			(hide yes)
@@
 			)
 		)
-		(property "Footprint" "Library:SOT-89_3MC_MCH"
+		(property "Footprint" "Package_TO_SOT_SMD:SOT-89-3"
 			(at 132.08 85.09 0)
 			(hide yes)
@@
 			)
 		)
-		(property "Footprint" "Library:SOT-89_3MC_MCH"
+		(property "Footprint" "Package_TO_SOT_SMD:SOT-89-3"
 			(at 69.85 170.18 0)
 			(hide yes)
